Commit message: Add SLAM mapping: room world, casters, wheel axis fix, saved map

File: src/my_robot_description/urdf/my_robot.urdf (robot description, URDF)
Before this commit: robot my_robot, 4 links, 3 joints
Links:
- added link caster_front, mass 0.05; collision sphere radius=0.05; visual sphere radius=0.05
- added link caster_rear, mass 0.05; collision sphere radius=0.05; visual sphere radius=0.05
Joints:
- added joint caster_front_joint: type fixed, parent base_link, child caster_front, origin xyz=0.15 0 -0.045 rpy=0 0 0
- added joint caster_rear_joint: type fixed, parent base_link, child caster_rear, origin xyz=-0.15 0 -0.045 rpy=0 0 0
- joint left_wheel_joint: axis 0 0 1 -> 0 0 -1
- joint right_wheel_joint: axis 0 0 1 -> 0 0 -1
