Commit message: Aim /scan by shrinking caster clearance to 3.5 mm
The caster clearance and the LiDAR beam elevation are two independently
reasonable decisions that nothing documents as coupled. The robot rests
nose-down on the front caster (the LiDAR's 0.3 kg at x=+0.12 puts the centre
of mass 5.6 mm ahead of the wheel axle), so the resting pitch subtracts
directly from the +1.000 deg beam. Their sum is where /scan actually points.

At the original 5.0 mm clearance that sum was -0.909 deg, putting the floor
intersection at 11.40 m inside a room whose diagonal is 12.806 m. The critical
clearance is 4.741 mm, so the design met its own requirement by 0.259 mm.

Drop the clearance to 3.5 mm (caster joint z -0.045 -> -0.0465). Resting pitch
falls 1.909 -> 1.337 deg, net /scan elevation -0.909 -> -0.337 deg, and the
floor intersection moves to 31.0 m -- past the sensor's own 30 m range limit,
so floor returns are impossible rather than unlikely.

Verified against a headless sim: measured resting pitch 1.33659 deg against
1.33666 deg predicted, 0.005 % off; chassis height 0.099986 m.

Rejected the intuitive fix. Moving the LiDAR onto the wheel axle would zero the
mass offset and let the robot rest level, but a robot balanced exactly on its
wheel line is in neutral equilibrium and would tip onto whichever caster the
landing noise favoured -- trading a deterministic tilt for a nondeterministic
one. Keeping the mass forward and shrinking the travel keeps it repeatable.

A descending beam is deliberate over an ascending one: an ascending beam stops
reporting low obstacles beyond some range, which for Nav2 is a collision.

Also correct a claim this file made in both READMEs. The platform's 11.8 %
hollow outline was attributed to the beam passing over it beyond 3.72 m,
computed from an assumed +1 deg upward tilt -- but the net elevation points
down, so the beam cannot clear a 0.25 m obstacle at any range. The measurement
is real; the explanation was not, and the perimeter-only account that replaces
it does not explain box1 at 50.6 %. Marked unresolved rather than patched.

maps/my_map.pgm and demo_map.gif were both recorded at the old -0.909 deg
geometry; flagged for regeneration before Nav2 localizes against them.

Co-Authored-By: Claude Opus 5 <noreply@anthropic.com>

File: src/my_robot_description/urdf/my_robot.urdf (robot description, URDF)
Before this commit: robot my_robot, 6 links, 5 joints
Joints:
- joint caster_front_joint: origin xyz=0.15 0 -0.045 rpy=0 0 0 -> xyz=0.15 0 -0.0465 rpy=0 0 0
- joint caster_rear_joint: origin xyz=-0.15 0 -0.045 rpy=0 0 0 -> xyz=-0.15 0 -0.0465 rpy=0 0 0
